Commit message: Update omni control and models

File: rbeken_description/robots/rbeken_mecanum_3f.urdf.xacro (robot description, xacro)
@@ -1,142 +1,157 @@
 <?xml version="1.0"?>
 <robot name="rbeken" xmlns:xacro="http://www.ros.org/wiki/xacro">
-	<!-- ***************** -->
-	<!-- Imported elements -->
-	<!-- ***************** -->
-	<!-- First we import all posible elements defined in the urdf.xacro files. All these elements are defined as macro:xacros -->
-	<!-- Import RB-Eken base elements -->
-	<xacro:include filename="$(find rbeken_description)/urdf/bases/rbeken_base.urdf.xacro" />
-	<!-- Import RB-Eken structures-->
-	<xacro:include filename="$(find rbeken_description)/urdf/structures/rbeken_gps_support.urdf.xacro" />
-	<!-- Import RB-Eken wheels -->
-	<xacro:include filename="$(find rbeken_description)/urdf/wheels/mecanum_wheel.urdf.xacro" />
-	<xacro:include filename="$(find rbeken_description)/urdf/structures/rbeken_laser_support.urdf.xacro" />
-	<!-- Import all available sensors -->
-	<xacro:include filename="$(find robotnik_sensors)/urdf/all_sensors.urdf.xacro" />
-	<xacro:property name="PI" value="3.1415926535897931"/>
-	<!-- Include force sensor description -->
-	<xacro:include filename="$(find rbeken_description)/urdf/robotiq_force_torque_sensor/robotiq_fts300.urdf.xacro" />
-	<!-- Include gripper description -->
-	<xacro:include filename="$(find rbeken_description)/urdf/robotiq_s/s-model_articulated_macro.xacro" />
-	<!-- Include UR-10 ARM -->
-	<xacro:include filename="$(find ur_description)/urdf/ur10.urdf.xacro" />
-		<!-- Wheel parameters -->
-	<xacro:property name="wheel_offset_x" value="0.26" />    <!-- x,y,z in translation from base_link to the center of the wheel -->
-	<xacro:property name="wheel_offset_y" value="0.295" />
-	<xacro:property name="wheel_offset_z" value="0.0" />
-	<xacro:property name="front_laser_offset_x" value="0.490"/>
-	<xacro:property name="front_laser_offset_y" value="-0.300"/>
-	<xacro:property name="front_laser_offset_z" value="0.2663"/>
- 	<xacro:property name="front_laser_offset_roll" value="${PI}"/>
-	<xacro:property name="front_laser_offset_pitch" value="0.0"/>
-	<xacro:property name="front_laser_offset_yaw" value="${PI/4}"/>
-	<xacro:property name="rear_laser_offset_x" value="-0.490"/>
-	<xacro:property name="rear_laser_offset_y" value="0.300"/>
-	<xacro:property name="rear_laser_offset_z" value="0.2663"/>
-	<xacro:property name="rear_laser_offset_roll" value="${PI}"/>
-	<xacro:property name="rear_laser_offset_yaw" value="${PI*4/4}"/>
-	<xacro:property name="front_laser_support_offset_x" value="0.345"/>
-	<xacro:property name="front_laser_support_offset_y" value="-0.300"/>
-	<xacro:property name="front_laser_support_offset_z" value="0.4085"/>
-	<xacro:property name="front_laser_support_offset_yaw" value="0"/>
-	<xacro:property name="rear_laser_support_offset_x" value="-0.345"/>
-	<xacro:property name="rear_laser_support_offset_y" value="0.300"/>
-	<xacro:property name="rear_laser_support_offset_z" value="0.4085"/>
- 	<xacro:property name="rear_laser_support_offset_yaw" value="${PI}"/>
-	<xacro:property name="front_ptz_camera_offset_x" value="0.41625"/>
-	<xacro:property name="front_ptz_camera_offset_y" value="0.0"/>
-	<xacro:property name="front_ptz_camera_offset_z" value="0.5043"/>
- 	<xacro:property name="front_ptz_camera_offset_roll" value="${PI}"/>
-	<xacro:property name="front_ptz_camera_offset_pitch" value="-0.6435029"/>
-	<xacro:property name="front_ptz_camera_offset_yaw" value="0.0"/>
-	<!--xacro:property name="rear_ptz_camera_offset_x" value="-0.308"/>
-	<xacro:property name="rear_ptz_camera_offset_y" value="-0.141"/>
-	<xacro:property name="rear_ptz_camera_offset_z" value="0.195"/-->
-	<xacro:property name="imu_offset_x" value="-0.384"/>
-	<xacro:property name="imu_offset_y" value="0.0"/>
-	<xacro:property name="imu_offset_z" value="0.4055"/>
-	<!--xacro:property name="front_rgbd_camera_offset_x" value="0.324"/>
-	<xacro:property name="front_rgbd_camera_offset_y" value="0.012"/>
-	<xacro:property name="front_rgbd_camera_offset_z" value="0.230"/-->
-	<xacro:property name="gps_offset_x" value="-0.540"/>
-	<xacro:property name="gps_offset_y" value="0.0"/>
-	<xacro:property name="gps_offset_z" value="0.898"/>
-	<!-- Flag to select the high or low quality model -->
-	<xacro:property name="hq" value="true" />
-	<xacro:arg name="prefix" default="rbeken_"/>
-	<xacro:arg name="ros_planar_move_plugin" default="false"/>
+    <!-- ***************** -->
+    <!-- Imported elements -->
+    <!-- ***************** -->
+    <!-- First we import all posible elements defined in the urdf.xacro files. All these elements are defined as macro:xacros -->
+    <!-- Import RB-Eken base elements -->
+    <xacro:include filename="$(find rbeken_description)/urdf/bases/rbeken_base.urdf.xacro" />
+    <!-- Import RB-Eken structures-->
+    <xacro:include filename="$(find rbeken_description)/urdf/structures/rbeken_gps_support.urdf.xacro" />
+    <!-- Import RB-Eken wheels -->
+    <xacro:include filename="$(find rbeken_description)/urdf/wheels/mecanum_wheel.urdf.xacro" />
+    <xacro:include filename="$(find rbeken_description)/urdf/structures/rbeken_laser_support.urdf.xacro" />
+    <!-- Import all available sensors -->
+    <xacro:include filename="$(find robotnik_sensors)/urdf/all_sensors.urdf.xacro" />
+    <xacro:property name="PI" value="3.1415926535897931"/>
+    <!-- Include force sensor description -->
+    <xacro:include filename="$(find rbeken_description)/urdf/robotiq_force_torque_sensor/robotiq_fts300.urdf.xacro" />
+    <!-- Include gripper description -->
+    <xacro:include filename="$(find rbeken_description)/urdf/robotiq_s/s-model_articulated_macro.xacro" />
+    <!-- Include UR-10 ARM -->
+    <xacro:include filename="$(find ur_description)/urdf/ur10.urdf.xacro" />
+        <!-- Wheel parameters -->
+    <xacro:property name="wheel_offset_x" value="0.26" />    <!-- x,y,z in translation from base_link to the center of the wheel -->
+    <xacro:property name="wheel_offset_y" value="0.295" />
+    <xacro:property name="wheel_offset_z" value="0.0" />
+    <xacro:property name="front_laser_offset_x" value="0.490"/>
+    <xacro:property name="front_laser_offset_y" value="-0.300"/>
+    <xacro:property name="front_laser_offset_z" value="0.2663"/>
+     <xacro:property name="front_laser_offset_roll" value="${PI}"/>
+    <xacro:property name="front_laser_offset_pitch" value="0.0"/>
+    <xacro:property name="front_laser_offset_yaw" value="${-PI/4}"/>
+    <xacro:property name="rear_laser_offset_x" value="-0.490"/>
+    <xacro:property name="rear_laser_offset_y" value="0.300"/>
+    <xacro:property name="rear_laser_offset_z" value="0.2663"/>
+    <xacro:property name="rear_laser_offset_roll" value="${PI}"/>
+    <xacro:property name="rear_laser_offset_yaw" value="${3*PI/4}"/>
+    <xacro:property name="front_laser_support_offset_x" value="0.345"/>
+    <xacro:property name="front_laser_support_offset_y" value="-0.300"/>
+    <xacro:property name="front_laser_support_offset_z" value="0.4085"/>
+    <xacro:property name="front_laser_support_offset_yaw" value="0"/>
+    <xacro:property name="rear_laser_support_offset_x" value="-0.345"/>
+    <xacro:property name="rear_laser_support_offset_y" value="0.300"/>
+    <xacro:property name="rear_laser_support_offset_z" value="0.4085"/>
+    <xacro:property name="rear_laser_support_offset_yaw" value="${PI}"/>
+    <xacro:property name="front_ptz_camera_offset_x" value="0.41625"/>
+    <xacro:property name="front_ptz_camera_offset_y" value="0.0"/>
+    <xacro:property name="front_ptz_camera_offset_z" value="0.5043"/>
+    <xacro:property name="front_ptz_camera_offset_roll" value="${PI}"/>
+    <xacro:property name="front_ptz_camera_offset_pitch" value="-0.6435029"/>
+    <xacro:property name="front_ptz_camera_offset_yaw" value="0.0"/>
+    <!--xacro:property name="rear_ptz_camera_offset_x" value="-0.308"/>
+    <xacro:property name="rear_ptz_camera_offset_y" value="-0.141"/>
+    <xacro:property name="rear_ptz_camera_offset_z" value="0.195"/-->
+    <xacro:property name="imu_offset_x" value="-0.384"/>
+    <xacro:property name="imu_offset_y" value="0.0"/>
+    <xacro:property name="imu_offset_z" value="0.4055"/>
+    <!--xacro:property name="front_rgbd_camera_offset_x" value="0.324"/>
+    <xacro:property name="front_rgbd_camera_offset_y" value="0.012"/>
+    <xacro:property name="front_rgbd_camera_offset_z" value="0.230"/-->
+    <xacro:property name="gps_offset_x" value="-0.540"/>
+    <xacro:property name="gps_offset_y" value="0.0"/>
+    <xacro:property name="gps_offset_z" value="0.898"/>
+    <!-- Flag to select the high or low quality model -->
+    <xacro:property name="hq" value="true" />
+    <xacro:arg name="prefix" default="rbeken_"/>
+    <xacro:arg name="ros_planar_move_plugin" default="false"/>
     <xacro:macro name="rbeken" params="prefix publish_bf hq">
-		<!-- *************** -->
-		<!-- Robots Elements -->
-		<!-- *************** -->
-		<!-- Here we create the robot elements using the xacro:macros imported at the beggining of this file -->
-		<!-- RB-Eken base -->
-		<xacro:rbeken_base prefix="$(arg prefix)" publish_bf="true" hq="${hq}" />
-		<xacro:omni_wheel prefix="$(arg prefix)front_right" parent="$(arg prefix)base_link" reflect="true" hq="${hq}">
-			<origin xyz="${wheel_offset_x} -${wheel_offset_y} ${wheel_offset_z}" rpy="0 0 0"/>
-		</xacro:omni_wheel>
-		<xacro:omni_wheel prefix="$(arg prefix)front_left" parent="$(arg prefix)base_link" reflect="false" hq="${hq}">
-			<origin xyz="${wheel_offset_x} ${wheel_offset_y} ${wheel_offset_z}" rpy="0 0 0"/>
-		</xacro:omni_wheel>
-		<xacro:omni_wheel prefix="$(arg prefix)back_left" parent="$(arg prefix)base_link" reflect="true" hq="${hq}">
-			<origin xyz="-${wheel_offset_x} ${wheel_offset_y} ${wheel_offset_z}" rpy="0 0 0"/>
-		</xacro:omni_wheel>
-		<xacro:omni_wheel prefix="$(arg prefix)back_right" parent="$(arg prefix)base_link" reflect="false" hq="${hq}">
-			<origin xyz="-${wheel_offset_x} -${wheel_offset_y} ${wheel_offset_z}" rpy="0 0 0"/>
-		</xacro:omni_wheel>
+        <!-- *************** -->
+        <!-- Robots Elements -->
+        <!-- *************** -->
+        <!-- Here we create the robot elements using the xacro:macros imported at the beggining of this file -->
+        <!-- RB-Eken base -->
+        <xacro:rbeken_base prefix="$(arg prefix)" publish_bf="true" hq="${hq}" />
+        <xacro:omni_wheel prefix="$(arg prefix)front_right" parent="$(arg prefix)base_link" reflect="true" hq="${hq}">
+            <origin xyz="${wheel_offset_x} -${wheel_offset_y} ${wheel_offset_z}" rpy="0 0 0"/>
+        </xacro:omni_wheel>
+        <xacro:omni_wheel prefix="$(arg prefix)front_left" parent="$(arg prefix)base_link" reflect="false" hq="${hq}">
+            <origin xyz="${wheel_offset_x} ${wheel_offset_y} ${wheel_offset_z}" rpy="0 0 0"/>
+        </xacro:omni_wheel>
+        <xacro:omni_wheel prefix="$(arg prefix)back_left" parent="$(arg prefix)base_link" reflect="true" hq="${hq}">
+            <origin xyz="-${wheel_offset_x} ${wheel_offset_y} ${wheel_offset_z}" rpy="0 0 0"/>
+        </xacro:omni_wheel>
+        <xacro:omni_wheel prefix="$(arg prefix)back_right" parent="$(arg prefix)base_link" reflect="false" hq="${hq}">
+            <origin xyz="-${wheel_offset_x} -${wheel_offset_y} ${wheel_offset_z}" rpy="0 0 0"/>
+        </xacro:omni_wheel>
         <!-- IMU -->
-		<xacro:sensor_imu_hector prefix="$(arg prefix)imu" parent="$(arg prefix)base_link">
-			<origin xyz="${imu_offset_x} ${imu_offset_y} ${imu_offset_z}" rpy="0 0 0"/>
-		</xacro:sensor_imu_hector>
-		<!-- Structures -->
-		<xacro:laser_support prefix="$(arg prefix)front_laser_structure" parent="$(arg prefix)base_link">
-			<origin xyz="${front_laser_support_offset_x} ${front_laser_support_offset_y} ${front_laser_support_offset_z}" rpy="0 0 ${front_laser_support_offset_yaw}" />
-		</xacro:laser_support>
-		<xacro:laser_support prefix="$(arg prefix)rear_laser_structure" parent="$(arg prefix)base_link">
-			<origin xyz="${rear_laser_support_offset_x} ${rear_laser_support_offset_y} ${rear_laser_support_offset_z}" rpy="0 0 ${rear_laser_support_offset_yaw}" />
-		</xacro:laser_support>
-		<!-- SENSORS -->
-		<xacro:sensor_sick_s300 prefix="$(arg prefix)front_laser" parent="$(arg prefix)base_link" prefix_topic="front_laser">
-			<origin xyz="${front_laser_offset_x} ${front_laser_offset_y} ${front_laser_offset_z}" rpy="${front_laser_offset_roll} ${front_laser_offset_pitch} ${front_laser_offset_yaw}"/>
-		</xacro:sensor_sick_s300>
-		<xacro:sensor_sick_s300 prefix="$(arg prefix)rear_laser" parent="$(arg prefix)base_link" prefix_topic="rear_laser">
-			<origin xyz="${rear_laser_offset_x} ${rear_laser_offset_y} ${rear_laser_offset_z}" rpy="${rear_laser_offset_roll} 0 ${rear_laser_offset_yaw}"/>
-		</xacro:sensor_sick_s300>
-		<xacro:sensor_axis_m5525 prefix="$(arg prefix)front_ptz_camera" parent="$(arg prefix)base_link">
-			<origin xyz="${front_ptz_camera_offset_x} ${front_ptz_camera_offset_y} ${front_ptz_camera_offset_z}" rpy="${front_ptz_camera_offset_roll} ${front_ptz_camera_offset_pitch} ${front_ptz_camera_offset_yaw}"/>
-		</xacro:sensor_axis_m5525>
-		<!-- GPS -->
-		<!--xacro:rbeken_gps_support prefix="$(arg prefix)gps_support" parent="$(arg prefix)base_link">
-				<origin xyz="${gps_offset_x} ${gps_offset_y} ${gps_offset_z}"/>
-		</xacro:rbeken_gps_support-->
-		<xacro:sensor_gps prefix="$(arg prefix)gps" parent="$(arg prefix)base_link">
-				<origin xyz="${gps_offset_x} ${gps_offset_y} ${gps_offset_z}"/>
-		</xacro:sensor_gps>
-			<!-- ROBOTIQ SENSOR -->
-		<xacro:robotiq_fts300 prefix="$(arg prefix)sensor_" parent="$(arg prefix)ur10_ee_link">
-			<origin xyz="0.0 0 0" rpy="0 -1.57 ${pi}"/>
-		</xacro:robotiq_fts300>
-		<!-- ROBOTIQ 3f GRIPPER -->
-		<xacro:s-model_articulated prefix="$(arg prefix)">
-		</xacro:s-model_articulated>
-		<!-- UR-10 ARM -->
-		<xacro:ur10_robot prefix="$(arg prefix)ur10_" joint_limited="true"
-			shoulder_pan_lower_limit="${-pi}" shoulder_pan_upper_limit="${pi}"
-			wrist_3_lower_limit="${-pi}" wrist_3_upper_limit="${pi}">
-		</xacro:ur10_robot>
-		<joint name="$(arg prefix)ur10_arm_base_joint" type="fixed">
-		  <origin xyz="0.215 0 0.5885" rpy="0 0 3.14"/>
-		  <parent link="$(arg prefix)base_link" />
-		  <child link="$(arg prefix)ur10_base_link" />
-		</joint>
-		<joint name="$(arg prefix)palm_joint" type="fixed">
-		  <origin xyz="0 0 0.05" rpy="1.57 0 ${pi*4/3}"/>
-		  <parent link="$(arg prefix)sensor_fts_toolside" />
-		  <child link="$(arg prefix)palm" />
-		</joint>
+        <xacro:sensor_imu_hector prefix="$(arg prefix)imu" parent="$(arg prefix)base_link">
+            <origin xyz="${imu_offset_x} ${imu_offset_y} ${imu_offset_z}" rpy="0 0 0"/>
+        </xacro:sensor_imu_hector>
+        <!-- Structures -->
+        <xacro:laser_support prefix="$(arg prefix)front_laser_structure" parent="$(arg prefix)base_link">
+            <origin xyz="${front_laser_support_offset_x} ${front_laser_support_offset_y} ${front_laser_support_offset_z}" rpy="0 0 ${front_laser_support_offset_yaw}" />
+        </xacro:laser_support>
+        <xacro:laser_support prefix="$(arg prefix)rear_laser_structure" parent="$(arg prefix)base_link">
+            <origin xyz="${rear_laser_support_offset_x} ${rear_laser_support_offset_y} ${rear_laser_support_offset_z}" rpy="0 0 ${rear_laser_support_offset_yaw}" />
+        </xacro:laser_support>
+        <!-- SENSORS -->
+        <xacro:sensor_sick_s300 prefix="$(arg prefix)front_laser" parent="$(arg prefix)base_link" prefix_topic="front_laser">
+            <origin xyz="${front_laser_offset_x} ${front_laser_offset_y} ${front_laser_offset_z}" rpy="${front_laser_offset_roll} ${front_laser_offset_pitch} ${front_laser_offset_yaw}"/>
+        </xacro:sensor_sick_s300>
+        <xacro:sensor_sick_s300 prefix="$(arg prefix)rear_laser" parent="$(arg prefix)base_link" prefix_topic="rear_laser">
+            <origin xyz="${rear_laser_offset_x} ${rear_laser_offset_y} ${rear_laser_offset_z}" rpy="${rear_laser_offset_roll} 0 ${rear_laser_offset_yaw}"/>
+        </xacro:sensor_sick_s300>
+        <xacro:sensor_axis_m5525 prefix="$(arg prefix)front_ptz_camera" parent="$(arg prefix)base_link" prefix_topic="front_ptz_camera">
+            <origin xyz="${front_ptz_camera_offset_x} ${front_ptz_camera_offset_y} ${front_ptz_camera_offset_z}" rpy="${front_ptz_camera_offset_roll} ${front_ptz_camera_offset_pitch} ${front_ptz_camera_offset_yaw}"/>
+        </xacro:sensor_axis_m5525>
+        <!-- GPS -->
+        <xacro:rbeken_gps_support prefix="$(arg prefix)gps_support" parent="$(arg prefix)base_link">
+                <origin xyz="${gps_offset_x} ${gps_offset_y} ${gps_offset_z}"/>
+        </xacro:rbeken_gps_support>
+        <xacro:sensor_gps prefix="$(arg prefix)gps" parent="$(arg prefix)base_link">
+            <origin xyz="${gps_offset_x} ${gps_offset_y} ${gps_offset_z}"/>
+        </xacro:sensor_gps>
+            <!-- ROBOTIQ SENSOR -->
+        <xacro:robotiq_fts300 prefix="$(arg prefix)sensor_" parent="$(arg prefix)arm_ee_link">
+            <origin xyz="0.0 0 0" rpy="0 -1.57 ${pi}"/>
+        </xacro:robotiq_fts300>
+        <!-- ROBOTIQ 3f GRIPPER -->
+        <xacro:s-model_articulated prefix="$(arg prefix)">
+        </xacro:s-model_articulated>
+        <!-- UR-10 ARM -->
+        <xacro:if value="$(arg load_kinematics_file)">
+            <xacro:ur10_robot prefix="$(arg prefix)arm_" joint_limited="true"
+            shoulder_pan_lower_limit="${-pi}" shoulder_pan_upper_limit="${pi}"
+            wrist_3_lower_limit="${-pi}" wrist_3_upper_limit="${pi}"
+            kinematics_file="${load_yaml('$(find rbeken_control)/config/ur10_calibration.yaml')}">
+            </xacro:ur10_robot>
+            <joint name="$(arg prefix)arm_base_joint" type="fixed">
+                <origin xyz="0.215 0 0.5885" rpy="0 0 3.14"/>
+                <parent link="$(arg prefix)base_link" />
+                <child link="$(arg prefix)arm_base_link" />
+            </joint>
+        </xacro:if>
+        <!-- UR-10 ARM -->
+        <xacro:unless value="$(arg load_kinematics_file)">
+            <xacro:ur10_robot prefix="$(arg prefix)arm_" joint_limited="true"
+            shoulder_pan_lower_limit="${-pi}" shoulder_pan_upper_limit="${pi}"
+            wrist_3_lower_limit="${-pi}" wrist_3_upper_limit="${pi}">
+            </xacro:ur10_robot>
+            <joint name="$(arg prefix)arm_base_joint" type="fixed">
+                <origin xyz="0.215 0 0.5885" rpy="0 0 3.14"/>
+                <parent link="$(arg prefix)base_link" />
+                <child link="$(arg prefix)arm_base_link" />
+            </joint>
+        </xacro:unless>
+        <joint name="$(arg prefix)palm_joint" type="fixed">
+          <origin xyz="0 0 0.05" rpy="1.57 0 ${pi*4/3}"/>
+          <parent link="$(arg prefix)sensor_fts_toolside" />
+          <child link="$(arg prefix)palm" />
+        </joint>
    </xacro:macro>
    <xacro:ros_control/>
    <xacro:if value="$(arg ros_planar_move_plugin)">
-	   <xacro:omni_steering prefix="$(arg prefix)" publish_tf="false"/>
+       <xacro:omni_steering prefix="$(arg prefix)" publish_tf="true"/>
    </xacro:if>
    <xacro:rbeken prefix="$(arg prefix)" publish_bf="true" hq="true"/>

File: rbeken_description/robots/rbeken_rubber_3f.urdf.xacro (robot description, xacro)
@@ -103,5 +103,5 @@
             <origin xyz="${rear_laser_offset_x} ${rear_laser_offset_y} ${rear_laser_offset_z}" rpy="${rear_laser_offset_roll} 0 ${rear_laser_offset_yaw}"/>
         </xacro:sensor_sick_s300>
-        <xacro:sensor_axis_m5525 prefix="$(arg prefix)front_ptz_camera" parent="$(arg prefix)base_link">
+        <xacro:sensor_axis_m5525 prefix="$(arg prefix)front_ptz_camera" parent="$(arg prefix)base_link" prefix_topic="front_ptz_camera">
             <origin xyz="${front_ptz_camera_offset_x} ${front_ptz_camera_offset_y} ${front_ptz_camera_offset_z}" rpy="${front_ptz_camera_offset_roll} ${front_ptz_camera_offset_pitch} ${front_ptz_camera_offset_yaw}"/>
         </xacro:sensor_axis_m5525>
