Commit message: Updated urdfs

File: rbeken_description/robots/rbeken_rubber.urdf.xacro (robot description, xacro)
@@ -16,5 +16,5 @@
     <xacro:property name="PI" value="3.1415926535897931"/>
     <!-- Include UR-10 ARM -->
-    <xacro:include filename="$(find ur_description)/urdf/ur10.urdf.xacro" />
+    <!--xacro:include filename="$(find ur_description)/urdf/ur10.urdf.xacro" /-->
     <!-- Include force sensor description -->
     <xacro:include filename="$(find rbeken_description)/urdf/robotiq_force_torque_sensor/robotiq_fts300.urdf.xacro" />
@@ -43,12 +43,12 @@
     <xacro:property name="rear_laser_support_offset_y" value="0.300"/>
     <xacro:property name="rear_laser_support_offset_z" value="0.4935"/>
-     <xacro:property name="rear_laser_support_offset_yaw" value="${PI}"/>
+    <xacro:property name="rear_laser_support_offset_yaw" value="${PI}"/>
     <xacro:property name="front_ptz_camera_offset_x" value="0.41625"/>
     <xacro:property name="front_ptz_camera_offset_y" value="0.0"/>
     <xacro:property name="front_ptz_camera_offset_z" value="0.5043"/>
-     <xacro:property name="front_ptz_camera_offset_roll" value="${PI}"/>
+    <xacro:property name="front_ptz_camera_offset_roll" value="${PI}"/>
     <xacro:property name="front_ptz_camera_offset_pitch" value="-0.6435029"/>
     <xacro:property name="front_ptz_camera_offset_yaw" value="0.0"/>
-    <!--xacro:property name="rear_ptz_camera_offset_x" value="-0.308"/>
+   <!--xacro:property name="rear_ptz_camera_offset_x" value="-0.308"/>
     <xacro:property name="rear_ptz_camera_offset_y" value="-0.141"/>
     <xacro:property name="rear_ptz_camera_offset_z" value="0.195"/-->
@@ -62,5 +62,5 @@
     <xacro:property name="gps_offset_y" value="0.0"/>
     <xacro:property name="gps_offset_z" value="0.898"/>
-    <!-- Flag to select the high or low quality model -->
+     <!-- Flag to select the high or low quality model -->
     <xacro:property name="hq" value="true" />
     <xacro:arg name="prefix" default="rbeken_"/>
@@ -117,12 +117,17 @@
         </xacro:sensor_gps>
         <!-- ROBOTIQ SENSOR -->
+        <!--
         <xacro:robotiq_fts300 prefix="$(arg prefix)sensor_" parent="$(arg prefix)arm_ee_link">
             <origin xyz="0 0 0" rpy="0 -1.57 ${pi}"/>
         </xacro:robotiq_fts300>
+        -->
         <!-- ROBOTIQ 85 GRIPPER -->
+        <!--
         <xacro:robotiq_85_gripper prefix="$(arg prefix)gripper_" parent="$(arg prefix)sensor_fts_toolside">
             <origin xyz="0 0.0 0" rpy="0 -1.57 0"/>
         </xacro:robotiq_85_gripper>
+        -->
         <!-- UR-10 ARM -->
+        <!--
         <xacro:if value="$(arg load_kinematics_file)">
             <xacro:ur10_robot prefix="$(arg prefix)arm_" joint_limited="true"
@@ -137,5 +142,5 @@
             </joint>
         </xacro:if>
-        <!-- UR-10 ARM -->
+        <! UR-10 ARM
         <xacro:unless value="$(arg load_kinematics_file)">
             <xacro:ur10_robot prefix="$(arg prefix)arm_" joint_limited="true"
@@ -149,4 +154,5 @@
             </joint>
         </xacro:unless>
+        -->
     </xacro:macro>
     <xacro:ros_control/>

File: rbeken_description/urdf/bases/rbeken_base.urdf.xacro (robot description, xacro)
@@ -31,6 +31,5 @@
             <mass value="250.0" />
             <origin xyz="0 0 0.2525" />
-            <box_inertia m="250" x="0.95" y="0.43" z="0.675"/>
-            <!--inertia  ixx="1.391" ixy="0.004"  ixz="0.0"  iyy="6.853"  iyz="0.0"  izz="6.125" /-->
+            <xacro:box_inertia m="250" x="0.95" y="0.43" z="0.675"/>
         </inertial>
         <visual>

File: rbeken_description/urdf/robotiq_c2/robotiq_85_gripper.urdf.xacro (robot description, xacro)
@@ -19,5 +19,5 @@
         </geometry>
       </collision>
-      <inertial>
+      <intertial>
         <mass value="0.636951" />
         <origin xyz="0.0 0.0 0.0" />
@@ -25,5 +25,5 @@
              iyx = "0.000000" iyy = "0.001110" iyz = "0.000000"
              izx = "0.000000" izy = "0.000000" izz = "0.001171" />
-      </inertial>
+      </intertial>
     </link>
     <joint name="${prefix}left_knuckle_joint" type="continuous">
@@ -52,5 +52,5 @@
         </geometry>
       </collision>
-      <inertial>
+      <intertial>
         <mass value="0.018491" />
         <origin xyz="0.0 0.0 0.0" />
@@ -58,5 +58,5 @@
              iyx = "-0.000001" iyy = "0.000001" iyz = "0.000000"
              izx = "0.000000" izy = "0.000000" izz = "0.000010" />
-      </inertial>
+      </intertial>
     </link>
     <link name="${prefix}right_knuckle_link">
@@ -71,5 +71,5 @@
         </geometry>
       </collision>
-      <inertial>
+      <intertial>
         <mass value="0.018491" />
         <origin xyz="0.0 0.0 0.0" />
@@ -77,5 +77,5 @@
              iyx = "-0.000001" iyy = "0.000001" iyz = "0.000000"
              izx = "0.000000" izy = "0.000000" izz = "0.000010" />
-      </inertial>
+      </intertial>
     </link>
     <joint name="${prefix}left_finger_joint" type="fixed">
@@ -100,5 +100,5 @@
         </geometry>
       </collision>
-      <inertial>
+      <intertial>
         <mass value="0.027309" />
         <origin xyz="0.0 0.0 0.0" />
@@ -106,5 +106,5 @@
              iyx = "-0.000002" iyy = "0.000021" iyz = "0.000000"
              izx = "0.000000" izy = "0.000000" izz = "0.000020" />
-      </inertial>
+      </intertial>
     </link>
     <link name="${prefix}right_finger_link">
@@ -119,5 +119,5 @@
         </geometry>
       </collision>
-      <inertial>
+      <intertial>
         <mass value="0.027309" />
         <origin xyz="0.0 0.0 0.0" />
@@ -125,5 +125,5 @@
              iyx = "-0.000002" iyy = "0.000021" iyz = "0.000000"
              izx = "0.000000" izy = "0.000000" izz = "0.000020" />
-      </inertial>
+      </intertial>
     </link>
     <joint name="${prefix}left_inner_knuckle_joint" type="continuous">
@@ -152,5 +152,5 @@
         </geometry>
       </collision>
-      <inertial>
+      <intertial>
         <mass value="0.029951" />
         <origin xyz="0.0 0.0 0.0" />
@@ -158,5 +158,5 @@
              iyx = "0.000000" iyy = "0.000005" iyz = "0.000000"
              izx = "0.000000" izy = "0.000000" izz = "0.000035" />
-      </inertial>
+      </intertial>
     </link>
     <link name="${prefix}right_inner_knuckle_link">
@@ -171,5 +171,5 @@
         </geometry>
       </collision>
-      <inertial>
+      <intertial>
         <mass value="0.029951" />
         <origin xyz="0.0 0.0 0.0" />
@@ -177,5 +177,5 @@
              iyx = "0.000000" iyy = "0.000005" iyz = "0.000000"
              izx = "0.000000" izy = "0.000000" izz = "0.000035" />
-      </inertial>
+      </intertial>
     </link>
     <joint name="${prefix}left_finger_tip_joint" type="continuous">
@@ -204,5 +204,5 @@
         </geometry>
       </collision>
-      <inertial>
+      <intertial>
         <mass value="0.019555" />
         <origin xyz="0.0 0.0 0.0" />
@@ -210,5 +210,5 @@
              iyx = "0.000000" iyy = "0.000005" iyz = "0.000000"
              izx = "0.000000" izy = "0.000000" izz = "0.000006" />
-      </inertial>
+      </intertial>
     </link>
     <link name="${prefix}right_finger_tip_link">
@@ -223,5 +223,5 @@
         </geometry>
       </collision>
-      <inertial>
+      <intertial>
         <mass value="0.019555" />
         <origin xyz="0.0 0.0 0.0" />
@@ -229,5 +229,5 @@
              iyx = "0.000000" iyy = "0.000005" iyz = "0.000000"
              izx = "0.000000" izy = "0.000000" izz = "0.000006" />
-      </inertial>
+      </intertial>
     </link>
     <!-- Improve grasping physics -->

File: rbeken_description/urdf/robotiq_c2/robotiq_85_gripper.xacro (robot description, xacro)
@@ -26,5 +26,5 @@
       </geometry>
     </collision>
-    <inertial>
+    <intertial>
       <mass value="1e2" />
       <origin xyz="0.0 0.0 0.0" />
@@ -32,5 +32,5 @@
            iyx = "0.000000" iyy = "0.000001" iyz = "0.000000"
            izx = "0.000000" izy = "0.000000" izz = "0.000001" />
-    </inertial>
+    </intertial>
   </link>
   <xacro:robotiq_85_gripper prefix="" parent="gripper_root_link" >

File: rbeken_description/urdf/robotiq_force_torque_sensor/robotiq_fts300.urdf.xacro (robot description, xacro)
@@ -10,9 +10,9 @@
         </joint>
         <link name="${prefix}fts_robotside">
-            <inertial>
+            <intertial>
                 <origin xyz="0 0 0.01875" rpy="0 0 0"/>
                 <mass value="0.65"/>
-                <inertia ixx="0.000661171875" ixy="0" ixz="0" iyy="0.000661171875" iyz="0" izz="0.00117" />
-            </inertial>
+                <intertia ixx="0.000661171875" ixy="0" ixz="0" iyy="0.000661171875" iyz="0" izz="0.00117" />
+            </intertial>
             <visual>
                 <origin xyz="0 0 0" rpy="0 0 0" />

File: rbeken_description/urdf/wheels/mecanum_wheel.urdf.xacro (robot description, xacro)
@@ -65,5 +65,5 @@
         <mass value="${wheel_mass}" />
         <origin xyz="0 0 0" />
-        <cylinder_inertia  m="${wheel_mass}" r="${wheel_radius}" h="${wheel_height}" />
+        <xacro:cylinder_inertia  m="${wheel_mass}" r="${wheel_radius}" h="${wheel_height}" />
       </inertial>
     </link>

File: rbeken_description/urdf/wheels/rubber_wheel.urdf.xacro (robot description, xacro)
@@ -52,5 +52,5 @@
         <mass value="${wheel_mass}" />
         <origin xyz="0 0 0" />
-        <cylinder_inertia  m="${wheel_mass}" r="${wheel_radius}" h="${wheel_height}" />
+        <xacro:cylinder_inertia  m="${wheel_mass}" r="${wheel_radius}" h="${wheel_height}" />
       </inertial>
     </link>

Commit message: Updates models

File: rbeken_description/robots/rbeken_rubber.urdf.xacro (robot description, xacro)
@@ -17,4 +17,5 @@
     <!-- Include UR-10 ARM -->
     <!--xacro:include filename="$(find ur_description)/urdf/ur10.urdf.xacro" /-->
+    <xacro:include filename="$(find ur_description)/urdf/inc/ur10e_macro.xacro" />
     <!-- Include force sensor description -->
     <xacro:include filename="$(find rbeken_description)/urdf/robotiq_force_torque_sensor/robotiq_fts300.urdf.xacro" />
@@ -62,4 +63,10 @@
     <xacro:property name="gps_offset_y" value="0.0"/>
     <xacro:property name="gps_offset_z" value="0.898"/>
+    <xacro:property name="arm_position_x" value="0.233"/>
+    <xacro:property name="arm_position_y" value="0"/>
+    <xacro:property name="arm_position_z" value="0.59250"/>
+    <xacro:property name="arm_orientation_r" value="0"/>
+    <xacro:property name="arm_orientation_p" value="0"/>
+    <xacro:property name="arm_orientation_y" value="0"/>
      <!-- Flag to select the high or low quality model -->
     <xacro:property name="hq" value="true" />
@@ -93,27 +100,27 @@
         </xacro:sensor_imu_hector>
         <!-- Structures -->
-        <xacro:laser_support prefix="$(arg prefix)front_laser_structure" parent="$(arg prefix)base_link">
+        <!--xacro:laser_support prefix="$(arg prefix)front_laser_structure" parent="$(arg prefix)base_link">
             <origin xyz="${front_laser_support_offset_x} ${front_laser_support_offset_y} ${front_laser_support_offset_z}" rpy="0 0 ${front_laser_support_offset_yaw}" />
-        </xacro:laser_support>
-        <xacro:laser_support prefix="$(arg prefix)rear_laser_structure" parent="$(arg prefix)base_link">
+        </xacro:laser_support-->
+        <!--xacro:laser_support prefix="$(arg prefix)rear_laser_structure" parent="$(arg prefix)base_link">
             <origin xyz="${rear_laser_support_offset_x} ${rear_laser_support_offset_y} ${rear_laser_support_offset_z}" rpy="0 0 ${rear_laser_support_offset_yaw}" />
-        </xacro:laser_support>
+        </xacro:laser_support-->
         <!-- SENSORS -->
-        <xacro:sensor_sick_s300 prefix="$(arg prefix)front_laser" parent="$(arg prefix)base_link" prefix_topic="front_laser" gpu="${gpu}">
+        <!--xacro:sensor_sick_s300 prefix="$(arg prefix)front_laser" parent="$(arg prefix)base_link" prefix_topic="front_laser" gpu="${gpu}">
             <origin xyz="${front_laser_offset_x} ${front_laser_offset_y} ${front_laser_offset_z}" rpy="${front_laser_offset_roll} ${front_laser_offset_pitch} ${front_laser_offset_yaw}"/>
-        </xacro:sensor_sick_s300>
-        <xacro:sensor_sick_s300 prefix="$(arg prefix)rear_laser" parent="$(arg prefix)base_link" prefix_topic="rear_laser" gpu="${gpu}">
+        </xacro:sensor_sick_s300-->
+        <!--xacro:sensor_sick_s300 prefix="$(arg prefix)rear_laser" parent="$(arg prefix)base_link" prefix_topic="rear_laser" gpu="${gpu}">
             <origin xyz="${rear_laser_offset_x} ${rear_laser_offset_y} ${rear_laser_offset_z}" rpy="${rear_laser_offset_roll} 0 ${rear_laser_offset_yaw}"/>
-        </xacro:sensor_sick_s300>
-        <xacro:sensor_axis_m5525 prefix="$(arg prefix)front_ptz_camera" parent="$(arg prefix)base_link" prefix_topic="front_ptz_camera">
+        </xacro:sensor_sick_s300-->
+        <!--xacro:sensor_axis_m5525 prefix="$(arg prefix)front_ptz_camera" parent="$(arg prefix)base_link" prefix_topic="front_ptz_camera">
             <origin xyz="${front_ptz_camera_offset_x} ${front_ptz_camera_offset_y} ${front_ptz_camera_offset_z}" rpy="${front_ptz_camera_offset_roll} ${front_ptz_camera_offset_pitch} ${front_ptz_camera_offset_yaw}"/>
-        </xacro:sensor_axis_m5525>
+        </xacro:sensor_axis_m5525-->
         <!-- GPS -->
-        <xacro:rbeken_gps_support prefix="$(arg prefix)gps_support" parent="$(arg prefix)base_link">
+        <!--xacro:rbeken_gps_support prefix="$(arg prefix)gps_support" parent="$(arg prefix)base_link">
             <origin xyz="${gps_offset_x} ${gps_offset_y} ${gps_offset_z}"/>
-        </xacro:rbeken_gps_support>
-        <xacro:sensor_gps prefix="$(arg prefix)gps" parent="$(arg prefix)base_link">
+        </xacro:rbeken_gps_support-->
+        <!--xacro:sensor_gps prefix="$(arg prefix)gps" parent="$(arg prefix)base_link">
             <origin xyz="${gps_offset_x} ${gps_offset_y} ${gps_offset_z}"/>
-        </xacro:sensor_gps>
+        </xacro:sensor_gps-->
         <!-- ROBOTIQ SENSOR -->
         <!--
@@ -141,18 +148,13 @@
                 <child link="$(arg prefix)arm_base_link" />
             </joint>
-        </xacro:if>
-        <! UR-10 ARM
-        <xacro:unless value="$(arg load_kinematics_file)">
-            <xacro:ur10_robot prefix="$(arg prefix)arm_" joint_limited="true"
-            shoulder_pan_lower_limit="${-pi}" shoulder_pan_upper_limit="${pi}"
-            wrist_3_lower_limit="${-pi}" wrist_3_upper_limit="${pi}">
-            </xacro:ur10_robot>
-            <joint name="$(arg prefix)arm_base_joint" type="fixed">
-                <origin xyz="0.215 0 0.5885" rpy="0 0 3.14"/>
-                <parent link="$(arg prefix)base_link" />
-                <child link="$(arg prefix)arm_base_link" />
-            </joint>
-        </xacro:unless>
-        -->
+        </xacro:if-->
+        <!-- UR-10e ARM -->
+        <!--xacro:ur10e_robot prefix="$(arg prefix)arm_">
+        </xacro:ur10e_robot>
+        <joint name="$(arg prefix)arm_base_joint" type="fixed">
+            <origin xyz="${arm_position_x} ${arm_position_y} ${arm_position_z}" rpy="${arm_orientation_r} ${arm_orientation_p} ${arm_orientation_y}"/>
+            <parent link="$(arg prefix)base_link" />
+            <child link="$(arg prefix)arm_base_link" />
+        </joint-->
     </xacro:macro>
     <xacro:ros_control/>

File: rbeken_description/urdf/bases/rbeken_base.urdf.xacro (robot description, xacro)
@@ -37,10 +37,10 @@
             <xacro:if value="${hq}">
             <geometry>
-                <mesh filename="package://rbeken_description/meshes/bases/rbeken_chasis.stl"/>
+                <mesh filename="package://rbeken_description/meshes/bases/rbeken_chasis_v2.stl"/>
             </geometry>
             </xacro:if>
             <xacro:unless value="${hq}">
             <geometry>
-                <mesh filename="package://rbeken_description/meshes/bases/rbeken_chasis.stl"/>
+                <mesh filename="package://rbeken_description/meshes/bases/rbeken_chasis_v2.stl"/>
             </geometry>
             </xacro:unless>
@@ -52,5 +52,5 @@
             <origin xyz="0 0 0" rpy="0 0 0 " />
             <geometry>
-                <mesh filename="package://rbeken_description/meshes/bases/rbeken_chasis.stl"/>
+                <mesh filename="package://rbeken_description/meshes/bases/rbeken_chasis_v2.stl"/>
             </geometry>
         </collision>

File: rbeken_description/urdf/wheels/rubber_wheel.urdf.xacro (robot description, xacro)
@@ -28,8 +28,8 @@
           <geometry>
 		<xacro:if value="${reflect}">
-			<mesh filename="package://rbeken_description/meshes/wheels/rbeken_rueda_goma.stl" />
+			<mesh filename="package://rbeken_description/meshes/wheels/rbeken_rubber_wheel_v2.stl" />
 		</xacro:if>
 		<xacro:unless value="${reflect}">
-			<mesh filename="package://rbeken_description/meshes/wheels/rbeken_rueda_goma.stl" />
+			<mesh filename="package://rbeken_description/meshes/wheels/rbeken_rubber_wheel_v2.stl" />
 		</xacro:unless>
           </geometry>
